File: ATU_transformer.kicad_sch (KiCad schematic)
At the start: 173 parts, among them J14 Conn_Coaxial, J16 Conn_Coaxial, J2 Conn_01x03, K1 G2R-1-E DC12, K10 G2R-1-E DC12, K11 G2R-1-E DC12, K12 G2R-1-E DC12, K13 G2R-1-E DC12, K14 G2R-1-E DC12, K15 G2R-1-E DC12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

Commit message: intermediate git, more traces to come
Parts:
- removed T1, T2: CST1, Transformer_SMD:Transformer_Coilcraft_CST1, symbol Transformer:CST1
- added T2: BN61-202, Amidon_Binocular:BN-61-202, symbol bn61-202:BN61-202
- R1, R2, R3, R4, R7, R8: footprint Resistor_SMD:R_1812_4532Metric_Pad1.30x3.40mm_HandSolder -> Resistor_SMD:R_2512_6332Metric_Pad1.40x3.35mm_HandSolder
Connections:
- net ATU_IN: now also T2.8
- net GND: now also T2.2, T2.6
- net at D2.2 (A), R2.2, R4.2: now also T2.4
- net at J14.1 (In): now also T2.1, T2.7
- net at D1.2 (A), R1.1, R3.1: now also T2.3, T2.5
Other:
- moved on the sheet: J14

Commit message: minor schematic mods
Other:
- note removed: "prendre des résistances de plus forte puissance"
Changed lines of the file:
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@@
     (stroke (width 0) (type default))
-  )
-  (text "prendre des résistances \nde plus forte puissance" (at 43.815 194.31 0)
-    (effects (font (size 2 2) (thickness 0.4) bold) (justify left bottom))
   )
   (text "??" (at 113.665 219.71 0)
